File: PowerSwitch/PowerSwitch.sch (KiCad schematic (older format))
At the start: 9 parts, among them J1 IN, J2 CTRL, J3 OUT, Q1 AO3400, Q2 AO3401

Commit message: Add KiBot script
Parts:
- Q1: JLC (none) -> C20917
- Q2: JLC (none) -> C15127
- R1, R3: JLC (none) -> C23212
- R2: JLC (none) -> C25819
- R4: JLC (none) -> C25804
Changed lines of the file:
@@
 EESchema Schematic File Version 4
-EELAYER 29 0
+EELAYER 30 0
 EELAYER END
 $Descr A4 11693 8268
@@
 F 2 "Resistor_SMD:R_0603_1608Metric_Pad1.05x0.95mm_HandSolder" V 2930 2100 50  0001 C CNN
 F 3 "~" H 3000 2100 50  0001 C CNN
+F 4 "C25819" V 3000 2100 50  0001 C CNN "JLC"
 	1    3000 2100
 	0    1    1    0
@@
 F 2 "Resistor_SMD:R_0603_1608Metric_Pad1.05x0.95mm_HandSolder" V 2280 2250 50  0001 C CNN
 F 3 "~" H 2350 2250 50  0001 C CNN
+F 4 "C23212" H 2350 2250 50  0001 C CNN "JLC"
 	1    2350 2250
 	-1   0    0    1
@@
 F 2 "Package_TO_SOT_SMD:SOT-23" H 3750 2200 50  0001 C CNN
 F 3 "~" H 3550 2100 50  0001 C CNN
+F 4 "C20917" H 3550 2100 50  0001 C CNN "JLC"
 	1    3550 2100
 	1    0    0    -1
@@
 F 2 "Package_TO_SOT_SMD:SOT-23" H 3850 1000 50  0001 C CNN
 F 3 "~" H 3650 900 50  0001 C CNN
+F 4 "C15127" V 3650 900 50  0001 C CNN "JLC"
 	1    3650 900
 	0    1    -1   0
@@
 F 2 "Resistor_SMD:R_0603_1608Metric_Pad1.05x0.95mm_HandSolder" V 3180 1150 50  0001 C CNN
 F 3 "~" H 3250 1150 50  0001 C CNN
+F 4 "C23212" V 3250 1150 50  0001 C CNN "JLC"
 	1    3250 1150
 	0    1    1    0
@@
 F 2 "Resistor_SMD:R_0603_1608Metric_Pad1.05x0.95mm_HandSolder" V 3580 1500 50  0001 C CNN
 F 3 "~" H 3650 1500 50  0001 C CNN
+F 4 "C25804" H 3650 1500 50  0001 C CNN "JLC"
 	1    3650 1500
 	-1   0    0    1
